Commit message: Using quadrotor mesh instead of building out of links

File: urdf/quadrotor.urdf.xacro (robot description, xacro)
@@ -1,155 +1,31 @@
 <?xml version="1.0"?>
 <robot xmlns:xacro="http://www.ros.org/wiki/xacro" name="roboarm">
-	<xacro:property name="base_mass" value="0.1"/>
-	<xacro:property name="base_height" value="0.02"/>
-	<xacro:property name="base_width" value="0.1"/>
-	<xacro:property name="base_length" value="0.1"/>
-	<xacro:property name="frame_mass" value="0.1"/>
-	<xacro:property name="frame_height" value="0.019"/>
-	<xacro:property name="frame_width" value="0.03"/>
-	<xacro:property name="frame_length" value="0.35"/>
-	<xacro:property name="rotor_mass" value="0.1"/>
-	<xacro:property name="rotor_height" value="0.02"/>
-	<xacro:property name="rotor_radius" value="0.04"/>
-	<link name="base_link">
+	<link name="quadrotor_link">
 		<inertial>
-			<mass value="${base_mass}"/>
-			<origin xyz="0 0 ${base_height/2}" rpy="0 0 0"/>
-			<inertia ixx="0.0"
+			<mass value="1.32"/>
+			<origin xyz="0 0 0.1825" rpy="0 0 0"/>
+			<inertia ixx="0.1"
 					 ixy="0.0"
 					 ixz="0.0"
-					 iyy="0.0"
+					 iyy="0.1"
 					 iyz="0.0"
-					 izz="0.0"/>
+					 izz="0.02"/>
 		</inertial>
-		<visual name="base_link_visual">
-			<origin xyz="0 0 ${base_height/2}" rpy="0 0 0"/>
+		<visual name="quadrotor_link_visual">
+			<origin xyz="0 0 0.1825" rpy="0 0 0"/>
 			<geometry>
-				<box size="${base_width} ${base_length} ${base_height}"/>
+				<mesh filename="package://cuda_swarm/meshes/quadrotor_base.dae"/>
 			</geometry>
 		</visual>
-		<collision name="base_collision_visual">
-			<origin xyz="0 0 ${base_height/2}" rpy="0 0 0"/>
+		<collision name="quadrotor_collision_visual">
+			<origin xyz="0 0 0.1825" rpy="0 0 0"/>
 			<geometry>
-				<box size="${base_width} ${base_length} ${base_height}"/>
+				<box size="0.8 0.8 0.365"/>
 			</geometry>
 		</collision>
 	</link>
-	<link name="frame_link">
-		<inertial>
-			<mass value="${frame_mass}"/>
-			<origin xyz="0 0 ${base_height/2}" rpy="0 0 0"/>
-			<inertia ixx="0.0"
-					 ixy="0.0"
-					 ixz="0.0"
-					 iyy="0.0"
-					 iyz="0.0"
-					 izz="0.0"/>
-		</inertial>
-		<visual name="frame_cw_link_visual">
-			<origin xyz="0 0 ${base_height/2}" rpy="0 0 ${-pi/4}"/>
-			<geometry>
-				<box size="${frame_length} ${frame_width} ${frame_height}"/>
-			</geometry>
-		</visual>
-		<visual name="frame_ccw_link_visual">
-			<origin xyz="0 0 ${base_height/2}" rpy="0 0 ${pi/4}"/>
-			<geometry>
-				<box size="${frame_length} ${frame_width} ${frame_height}"/>
-			</geometry>
-		</visual>
-		<collision name="frame_cw_link_collision">
-			<origin xyz="0 0 ${base_height/2}" rpy="0 0 ${-pi/4}"/>
-			<geometry>
-				<box size="${frame_length} ${frame_width} ${frame_height}"/>
-			</geometry>
-		</collision>
-		<collision name="frame_ccw_link_collision">
-			<origin xyz="0 0 ${base_height/2}" rpy="0 0 ${pi/4}"/>
-			<geometry>
-				<box size="${frame_length} ${frame_width} ${frame_height}"/>
-			</geometry>
-		</collision>
-	</link>
-	<link name="rotor_link">
-		<inertial>
-			<mass value="${rotor_mass}"/>
-			<origin xyz="0 0 ${base_height/2}" rpy="0 0 0"/>
-			<inertia ixx="0.0"
-					 ixy="0.0"
-					 ixz="0.0"
-					 iyy="0.0"
-					 iyz="0.0"
-					 izz="0.0"/>
-		</inertial>
-		<visual name="front_right_rotor_visual">
-			<origin xyz="${(0.5*frame_length-0.9*rotor_radius)*cos(pi/4)} ${(0.5*frame_length-0.9*rotor_radius)*sin(pi/4)} ${base_height/2}"/>
-			<geometry>
-				<cylinder length="${rotor_height}" radius="${rotor_radius}"/>
-			</geometry>
-		</visual>
-		<visual name="front_left_rotor_visual">
-			<origin xyz="${-(0.5*frame_length-0.9*rotor_radius)*cos(pi/4)} ${(0.5*frame_length-0.9*rotor_radius)*sin(pi/4)} ${base_height/2}"/>
-			<geometry>
-				<cylinder length="${rotor_height}" radius="${rotor_radius}"/>
-			</geometry>
-		</visual>
-		<visual name="back_right_rotor_visual">
-			<origin xyz="${(0.5*frame_length-0.9*rotor_radius)*cos(pi/4)} ${-(0.5*frame_length-0.9*rotor_radius)*sin(pi/4)} ${base_height/2}"/>
-			<geometry>
-				<cylinder length="${rotor_height}" radius="${rotor_radius}"/>
-			</geometry>
-		</visual>
-		<visual name="back_left_rotor_visual">
-			<origin xyz="${-(0.5*frame_length-0.9*rotor_radius)*cos(pi/4)} ${-(0.5*frame_length-0.9*rotor_radius)*sin(pi/4)} ${base_height/2}"/>
-			<geometry>
-				<cylinder length="${rotor_height}" radius="${rotor_radius}"/>
-			</geometry>
-		</visual>
-		<collision name="front_right_rotor_collision">
-			<origin xyz="${(0.5*frame_length-0.9*rotor_radius)*cos(pi/4)} ${(0.5*frame_length-0.9*rotor_radius)*sin(pi/4)} ${base_height/2}"/>
-			<geometry>
-				<cylinder length="${rotor_height}" radius="${rotor_radius}"/>
-			</geometry>
-		</collision>
-		<collision name="front_left_rotor_collision">
-			<origin xyz="${-(0.5*frame_length-0.9*rotor_radius)*cos(pi/4)} ${(0.5*frame_length-0.9*rotor_radius)*sin(pi/4)} ${base_height/2}"/>
-			<geometry>
-				<cylinder length="${rotor_height}" radius="${rotor_radius}"/>
-			</geometry>
-		</collision>
-		<collision name="back_right_rotor_collision">
-			<origin xyz="${(0.5*frame_length-0.9*rotor_radius)*cos(pi/4)} ${-(0.5*frame_length-0.9*rotor_radius)*sin(pi/4)} ${base_height/2}"/>
-			<geometry>
-				<cylinder length="${rotor_height}" radius="${rotor_radius}"/>
-			</geometry>
-		</collision>
-		<collision name="back_left_rotor_collision">
-			<origin xyz="${-(0.5*frame_length-0.9*rotor_radius)*cos(pi/4)} ${-(0.5*frame_length-0.9*rotor_radius)*sin(pi/4)} ${base_height/2}"/>
-			<geometry>
-				<cylinder length="${rotor_height}" radius="${rotor_radius}"/>
-			</geometry>
-		</collision>
-	</link>
-	<joint name="base_to_frame_fixed" type="fixed">
-		<parent link="base_link"/>
-		<child link="frame_link"/>
-	</joint>
-	<joint name="frame_to_rotor_fixed" type="fixed">
-		<parent link="frame_link"/>
-		<child link="rotor_link"/>
-	</joint>
 	<gazebo>
 		<static>False</static>
 		<plugin name="gazebo_ros_control" filename="libgazebo_ros_control.so"/>
 	</gazebo>
-	<gazebo reference="base_link">
-		<material>Gazebo/Black</material>
-	</gazebo>
-	<gazebo reference="frame_link">
-		<material>Gazebo/Red</material>
-	</gazebo>
-	<gazebo reference="rotor_link">
-		<material>Gazebo/Black</material>
-	</gazebo>
 </robot>
